File: PCB/PCB.kicad_sch (KiCad schematic)
At the start: 39 parts, among them J1 Conn_01x04_Pin, SW1 SW_Push, SW10 SW_Push, SW11 SW_Push, SW12 SW_Push, SW13 SW_Push, SW14 SW_Push, SW15 SW_Push, SW16 SW_Push, SW17 SW_Push, SW2 SW_Push, SW3 SW_Push, SW4 SW_Push, SW5 SW_Push, SW6 SW_Push, SW7 SW_Push, SW8 SW_Push, SW9 SW_Push, U1 XIAO-RP2040-DIP

Commit message: why was this not in previous commit?
Parts:
- removed J1: Conn_01x04_Pin, Number-Pad:SSD1306-0.91-OLED-4pin-128x32, symbol Connector:Conn_01x04_Pin
Connections:
- net +3V3: no longer names the net of U1.12 (3V3_OUT)
- net SCL: no longer names the net of U1.10 (D9)
- net SDA: no longer names the net of U1.11 (D10)
