File: PCB/PCB.kicad_pcb (KiCad board)
At the start: 2 copper layers, 77.6 x 116.7 mm, 39 parts, among them J1 Conn_01x04_Pin, SW1 SW_Push, SW10 SW_Push, SW11 SW_Push, SW12 SW_Push, SW13 SW_Push, SW14 SW_Push, SW15 SW_Push, SW16 SW_Push, SW17 SW_Push, SW2 SW_Push, SW3 SW_Push, SW4 SW_Push, SW5 SW_Push, SW6 SW_Push, SW7 SW_Push, SW8 SW_Push, SW9 SW_Push, U1 XIAO-RP2040-DIP

Commit message: why was this not in previous commit?
Parts:
- removed J1: Conn_01x04_Pin, Number-Pad:SSD1306-0.91-OLED-4pin-128x32
- added G***: LOGO, Polyglot_footprints:40mm_Sabhya, F.Cu at (150.8, 67.2)
Connections:
- U1 pad 10: SCL -> unconnected-(U1-D9-Pad10)
- U1 pad 11: SDA -> unconnected-(U1-D10-Pad11)
- U1 pad 12: +3V3 -> unconnected-(U1-3V3_OUT-Pad12)
Routing:
- net SCL: track 27.8 -> 0.00 mm
- net +3V3: track 25.4 -> 0.00 mm
- net SDA: track 20.7 -> 0.00 mm
- added copper zone on B.Cu, net (none)
- added copper zone on F.Cu, net (none)
- removed copper zone on B.Cu, net GND
- removed copper zone on F.Cu, net GND

Commit message: smth
Parts:
- moved D11 16.3 mm to (141.8, 118.4)
- moved D3 16.3 mm to (155.1, 74.6)
- moved D8 16.3 mm to (160.8, 108.9)
- moved S8 16.3 mm to (164.6, 99.4)
- moved SW11 16.3 mm to (145.6, 108.9)
- moved SW8 16.3 mm to (164.6, 99.4)
- moved D1 16.3 mm to (117.0, 74.6)
- moved D9 16.3 mm to (117.0, 112.7)
- moved SW9 16.3 mm to (107.5, 108.9)
- moved D10 16.3 mm to (136.0, 112.7)
- moved D2 16.3 mm to (136.0, 74.6)
- moved SW10 16.3 mm to (126.5, 108.9)
- moved D14 16.3 mm to (141.8, 137.4)
- moved D15 16.3 mm to (160.8, 147.0)
- moved D16 16.3 mm to (126.5, 150.8)
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